File: pixle.kicad_pcb (KiCad board)
At the start: 2 copper layers, 60.8 x 53.3 mm, 26 parts, among them J1 Barrel_Jack_MountingPin, M1 28BYJ-48, M2 28BYJ-48, M3 28BYJ-48, M4 28BYJ-48, SW1 PUSH_RESET, U1 ULN2003, U2 ULN2003, U3 ULN2003

Commit message: updated board
Parts:
- removed the REF** at (116.0, 76.6)
- removed the REF** at (116.5, 120.6)
- removed the REF** at (64.8, 120.3)
- removed the REF** at (64.8, 76.8)
- removed the U1 at (92.5, 85.8)
- added REF**: MountingHole_M3, pixle:MountingHole_M3, F.Cu at (107.8, 121.3)
- added REF**: MountingHole_M3, pixle:MountingHole_M3, F.Cu at (64.2, 121.3)
- added REF**: MountingHole_M3, pixle:MountingHole_M3, F.Cu at (99.2, 75.3)
- added REF**: MountingHole_M3, pixle:MountingHole_M3, F.Cu at (64.2, 75.3)
- added U0: ULN2003, Package_DIP:DIP-16_W7.62mm, F.Cu at (92.2, 81.5)
- moved PP1 60.8 mm to (71.0, 122.4), turned to 90 degrees
- moved I2C_0 55.9 mm to (76.7, 75.1), turned to 0 degrees
- moved I2C_1 47.5 mm to (87.0, 75.1), turned to 0 degrees
- moved LS3 41.4 mm to (114.4, 111.8), turned to 0 degrees
- moved C3 39.4 mm to (84.5, 120.2), turned to 270 degrees
- moved R1 39.1 mm to (72.2, 118.8), turned to 0 degrees
- moved SW1 35.7 mm to (119.0, 123.2)
- moved LS0 28.8 mm to (114.4, 87.8)
- moved M0 28.8 mm to (97.9, 87.8)
- moved C1 28.5 mm to (89.8, 122.9), turned to 180 degrees
- moved C0 27.6 mm to (87.2, 119.9), turned to 0 degrees
- moved M1 19.3 mm to (97.9, 95.8), turned to 0 degrees
- moved XO1 19.2 mm to (100.0, 121.4), turned to 180 degrees
- moved M2 14.8 mm to (97.9, 103.8), turned to 0 degrees
- moved LS1 14.8 mm to (114.4, 95.8), turned to 0 degrees
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- renumbered A1 to A, C2 to C0, I2C_1 to I2C_0, I2C_2 to I2C_1, J1 to J, LS1 to LS0, LS2 to LS1, LS3 to LS2, LS4 to LS3, M1 to M0, M2 to M1, M3 to M2, M4 to M3, U2 to U1, U3 to U2
Routing:
- net Net-(A1-Pad28): track 94.1 -> 22.9 mm
- net Net-(A1-Pad3): track 190.1 -> 120.5 mm
- net Net-(A1-Pad27): track 92.8 -> 24.8 mm
- net +5V: track 229.5 -> 162.9 mm
- net Net-(A1-Pad9): track 104.0 -> 55.2 mm
- net Net-(A1-Pad10): track 93.3 -> 58.9 mm
- net Net-(M1-Pad1): track 46.7 -> 15.3 mm
- net Net-(M2-Pad4): track 54.7 -> 27.5 mm
- net Net-(M2-Pad2): track 41.3 -> 15.2 mm
- net Net-(M2-Pad3): track 47.9 -> 21.9 mm
- net Net-(M2-Pad1): track 33.1 -> 9.16 mm
- net Net-(M4-Pad4): track 5.92 -> 26.7 mm
- net Net-(M3-Pad2): track 42.8 -> 23.6 mm
- net Net-(M1-Pad2): track 38.2 -> 20.9 mm
- net Net-(M3-Pad1): track 33.8 -> 17.9 mm
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Other:
- board size 60.8 x 53.3 mm -> 59.5 x 53.3 mm
