File: pixle.sch (KiCad schematic (older format))
At the start: 22 parts, among them J1 Barrel_Jack_MountingPin, M1 28BYJ-48, M2 28BYJ-48, M3 28BYJ-48, M4 28BYJ-48, SW1 PUSH_RESET, U1 ULN2003, U2 ULN2003, U3 ULN2003

Commit message: updated board
Parts:
- renumbered C2 to C1, C1 to C2, I2C_2 to I2C_1, I2C_1 to I2C_2
Connections:
- no-connect marks 0 -> 11
