File: pixel.kicad_pcb (KiCad board)
At the start: 2 copper layers, 59.5 x 53.3 mm, 26 parts, among them M0 28BYJ-48, M1 28BYJ-48, M2 28BYJ-48, M3 28BYJ-48, SW1 PUSH_RESET, U0 ULN2003, U1 ULN2003, U2 ULN2003

Commit message: renamed pixle to pixel
Parts:
- REF** (x4): footprint pixle:MountingHole_M3 -> pixel:MountingHole_M3
- SW1: footprint pixle:SW_PUSH_6mm_2pin -> pixel:SW_PUSH_6mm_2pin
Changed lines of the file:
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@@
     (add_net "Net-(M4-Pad4)")
   )
-  (module pixle:MountingHole_M3 (layer F.Cu)
+  (module pixel:MountingHole_M3 (layer F.Cu)
     (at 107.85 121.35)
     (descr "Mounting Hole 3.2mm, no annular, M3")
@@
     (pad 1 np_thru_hole circle (at 0 0) (size 3.2 3.2) (drill 3.2) (layers *.Cu *.Mask))
   )
-  (module pixle:MountingHole_M3 (layer F.Cu)
+  (module pixel:MountingHole_M3 (layer F.Cu)
     (at 64.15 121.35)
     (descr "Mounting Hole 3.2mm, no annular, M3")
@@
     (pad 1 np_thru_hole circle (at 0 0) (size 3.2 3.2) (drill 3.2) (layers *.Cu *.Mask))
   )
-  (module pixle:MountingHole_M3 (layer F.Cu)
+  (module pixel:MountingHole_M3 (layer F.Cu)
     (at 99.2 75.35)
     (descr "Mounting Hole 3.2mm, no annular, M3")
@@
     (pad 1 np_thru_hole circle (at 0 0) (size 3.2 3.2) (drill 3.2) (layers *.Cu *.Mask))
   )
-  (module pixle:MountingHole_M3 (layer F.Cu)
+  (module pixel:MountingHole_M3 (layer F.Cu)
     (at 64.15 75.35)
     (descr "Mounting Hole 3.2mm, no annular, M3")
@@
     )
   )
-  (module pixle:SW_PUSH_6mm_2pin (layer F.Cu)
+  (module pixel:SW_PUSH_6mm_2pin (layer F.Cu)
     (at 119 123.25 180)
     (descr https://www.omron.com/ecb/products/pdf/en-b3f.pdf)
