File: pixel.sch (KiCad schematic (older format))
At the start: 22 parts, among them J1 Barrel_Jack_MountingPin, M1 28BYJ-48, M2 28BYJ-48, M3 28BYJ-48, M4 28BYJ-48, SW1 PUSH_RESET, U1 ULN2003, U2 ULN2003, U3 ULN2003

Commit message: renamed pixle to pixel
Parts:
- A1: symbol pixle:ATmega328P-PU -> pixel:ATmega328P-PU
- I2C_1, I2C_2: symbol pixle:I2C -> pixel:I2C
- J1: symbol pixle:Barrel_Jack_MountingPin -> pixel:Barrel_Jack_MountingPin
- LS1, LS2, LS3, LS4: symbol pixle:Limit_Switch -> pixel:Limit_Switch
- M1, M2, M3, M4: symbol pixle:28BYJ-48 -> pixel:28BYJ-48
- PP1: symbol pixle:ProgramPort -> pixel:ProgramPort
- SW1: footprint pixle:SW_PUSH_6mm_2pin -> pixel:SW_PUSH_6mm_2pin
- U1, U2, U3: symbol pixle:ULN2003 -> pixel:ULN2003
Changed lines of the file:
@@
 $EndDescr
 $Comp
-L pixle:ULN2003 U3
+L pixel:ULN2003 U3
 U 1 1 60D72B6F
 P 8150 4300
@@
 $EndComp
 $Comp
-L pixle:ULN2003 U2
+L pixel:ULN2003 U2
 U 1 1 60DD8EF7
 P 8150 2050
@@
 	5800 3750 5650 3750
 $Comp
-L pixle:ULN2003 U1
+L pixel:ULN2003 U1
 U 1 1 60D75900
 P 3100 4100
@@
 $EndComp
 $Comp
-L pixle:28BYJ-48 M2
+L pixel:28BYJ-48 M2
 U 1 1 60DF70FB
 P 9450 1700
@@
 $EndComp
 $Comp
-L pixle:28BYJ-48 M3
+L pixel:28BYJ-48 M3
 U 1 1 60DF8B5A
 P 9450 3300
@@
 $EndComp
 $Comp
-L pixle:28BYJ-48 M4
+L pixel:28BYJ-48 M4
 U 1 1 60DF9646
 P 9450 4950
@@
 	2700 4050 2050 4050
 $Comp
-L pixle:28BYJ-48 M1
+L pixel:28BYJ-48 M1
 U 1 1 60DF9A92
 P 2000 3750
@@
 	7250 2400 7750 2400
 $Comp
-L pixle:ATmega328P-PU A1
+L pixel:ATmega328P-PU A1
 U 1 1 60D41184
 P 6400 3000
@@
 	5500 3650 4450 3650
 $Comp
-L pixle:Limit_Switch LS2
+L pixel:Limit_Switch LS2
 U 1 1 60F4A77E
 P 9950 2500
@@
 $EndComp
 $Comp
-L pixle:Limit_Switch LS3
+L pixel:Limit_Switch LS3
 U 1 1 60F4C901
 P 9950 4200
@@
 $EndComp
 $Comp
-L pixle:Limit_Switch LS4
+L pixel:Limit_Switch LS4
 U 1 1 60F4CD92
 P 9950 5650
@@
 Connection ~ 1500 3000
 $Comp
-L pixle:ProgramPort PP1
+L pixel:ProgramPort PP1
 U 1 1 60E0B971
 P 4800 2100
@@
 F 0 "SW1" H 6300 1785 50  0000 C CNN
 F 1 "PUSH_RESET" H 6300 1694 50  0000 C CNN
-F 2 "pixle:SW_PUSH_6mm_2pin" H 6300 1700 50  0001 C CNN
+F 2 "pixel:SW_PUSH_6mm_2pin" H 6300 1700 50  0001 C CNN
 F 3 "~" H 6300 1700 50  0001 C CNN
 	1    6300 1500
@@
 $EndComp
 $Comp
-L pixle:I2C I2C_2
+L pixel:I2C I2C_2
 U 1 1 60EB02D7
 P 7500 950
@@
 $EndComp
 $Comp
-L pixle:I2C I2C_1
+L pixel:I2C I2C_1
 U 1 1 60EB0F46
 P 7050 950
@@
 Connection ~ 7000 1150
 $Comp
-L pixle:Barrel_Jack_MountingPin J1
+L pixel:Barrel_Jack_MountingPin J1
 U 1 1 60F94B90
 P 1700 1600
@@
 $EndComp
 $Comp
-L pixle:Limit_Switch LS1
+L pixel:Limit_Switch LS1
 U 1 1 60F49BCC
 P 1700 3100
